File: Schematics/KiCAD/joytester.kicad_pcb (KiCad board)
At the start: 2 copper layers, 38 x 66 mm, 12 parts

Commit message: Cosmetic changed - added 3d components to 3d view
Other:
- board text added: "Copyright (C) 2018-2021 http://retro-commodore.eu"
- board text removed: "Copyright (C) 2018-2020 http://retro-commodore.eu"
